Commit message: 램프 배달물 0814 판으로 교체 — 볼록 분해와 glTF 색을 그대로 쓴다
새 배달물이 우리가 손으로 만들던 것을 직접 준다.
  drake/collisions/link_N/part_XX.obj   볼록 분해 (10/5/6 조각)
  drake/visuals/link_N_*_rgb.gltf       정점 색(COLOR_0) 이 든 glTF

  - 색이 비슷한 면끼리 쪼개 단색을 입히던 우회를 그만뒀다. Meshcat 의
    glTF 로더가 COLOR_0 을 그대로 그린다.
  - 볼록 분해도 배달물 것을 쓴다. 예전에는 삭제된 배달물에서 구운 캐시를
    재활용하고 있었다.
  - 부피·도심은 예전 배달물과 소수점까지 같다 (441.02 / 165.70 / 219.58
    cm^3). 같은 물체의 포장만 좋아진 것이다.

파지점을 도심에서 **실제로 물리는 자리** 로 바꿨다. 굽은 팔의 도심은 재료
안에 있어도 그 자리 단면의 중심은 아니라서, 죠를 오므리면 한쪽 패드가
10.5 mm 허공을 물었다 (파지점 근처 재료가 -11.7~+3.2 mm 인데 패드는
+-13.7 mm 에 있었다). 볼록 조각은 팔을 토막 낸 것이라 거의 원기둥이므로,
조각의 중심을 파지점으로, 최단 주축을 죠 방향으로, 최장 주축을 손목 축으로
쓴다. 폭은 조각 전체가 아니라 파지점 근처 30 mm 에서 잰다.

  link_3 part_00: 파지점 [0.254 0.409 0.088], 폭 17.6 mm
  개구 17.6 mm -> 패드 x = +-8.8 mm, 파지점 근처 재료 -8.3 ~ +9.3 mm

굽은 팔의 파지 방향은 좌표축에 나란하지 않으므로 Part.grasp_axis 가 축
번호 대신 단위벡터도 받도록 했다.

재검증: 램프 20/25 후보, 2 라운드, 오차 0.00~0.18%.
        3link 23/25, 2link 5/5, 진단 12/12.

Co-Authored-By: Claude Opus 5 <noreply@anthropic.com>

File: assets/desk_lamp_minimal_sim/drake/object.urdf (robot description, URDF)
Before this commit: robot object, 4 links, 3 joints
Links:
- link link_1: geometry collision mesh filename=collisions/link_1/part_00.obj; collision mesh filename=collisions/link_1/part_01.obj
- link link_2: geometry collision mesh filename=collisions/link_2/part_00.obj; collision mesh filename=collisions/link_2/part_01.obj
- link link_3: geometry collision mesh filename=collisions/link_3/part_00.obj; collision mesh filename=collisions/link_3/part_01.obj
