Commit message: 경로가 거꾸로 나오던 것을 고친다 — 순간이동의 진짜 원인
RRT-Connect 는 두 트리를 번갈아 키우느라 매 반복마다 a 와 b 를 맞바꾼다.
그래서 연결이 성사된 순간의 tree_a 가 출발 쪽이 아닐 수 있는데, 그걸 안
따지고 path_a + path_b 로 이어 붙이고 있었다. 결과는 **통째로 뒤집힌 경로**다.

계측이 그대로 말해 주었다.

  [진단] 경로가 어긋납니다: path[0]-start 134.2 deg, path[-1]-target 134.2 deg
  [로봇] 경고: 화면이 134.2 deg 건너뜁니다 (프레임 0)

두 값이 같다는 것은 path[0]=목표, path[-1]=출발 이라는 뜻이다. 그래서 로봇은
목표 자세로 순간이동한 뒤 거꾸로 되짚어 와 출발점에 멈췄다 — 각도 측정
자세에 애초에 도착하지 못했다. 시뮬레이션의 렌치는 팔 자세가 아니라 물체
각도와 중력 방향으로 계산되므로 숫자만 보면 멀쩡해 보였다.

트리 교대를 따라가는 깃발을 두고, 마지막에 시작점 거리로 한 번 더 확인한다.
44개 경로 전부 방향이 맞는다 (전에는 여러 개가 뒤집혀 있었다).

그리퍼 개구도 고쳤다. 각도를 rpy 에 구워 넣을 때 부호가 반대여서 오므리라고
할수록 벌어졌다 (19.4 mm 요청 -> 실제 116.5 mm). 축 회전을 제대로 곱하도록
바꿨고 요청값과 실제 간격이 소수점까지 맞는다.

감시 두 개를 붙였다: 프레임 사이 관절 도약(순간이동), 이동 중 최소 간격.
고친 뒤 순간이동 0건, 경로 어긋남 0건, 프레임 최대 0.54 deg,
이동 중 최소 간격 5.5~6.0 mm, 램프 2 라운드 오차 0.00~0.23%.

새 대화에서 이어받을 수 있도록 HANDOFF.md 를 추가했다.

Co-Authored-By: Claude Opus 5 <noreply@anthropic.com>

File: my_work/estimated_desklamp.urdf (robot description, URDF)
Before this commit: robot desklamp_estimated, 3 links, 2 joints
Links:
- link link_1: mass 0.084023 -> 0.084003
- link link_2: mass 0.396004 -> 0.396025
- link link_3: mass 0.082087 -> 0.082086
