Commit message: 실물 준비 — 여유 1cm, 물성 주입 URDF, 수동 파지, 각도 ±5도
전부 계측해서 확인했다.

여유 간격 6mm -> 10mm
  실물에는 모형에 없는 오차가 겹쳐 쌓인다 (손-눈 잔차, 자세 오차,
  파지점 어긋남 5mm, 스캔 형상 오차).

  고치다 보니 **10mm 를 요구해도 9mm 까지 파고들 수 있었다.** 계획기가
  문턱을 10% 낮춰 잡고 있었다 (PLANNER_MARGIN_RATIO). IK 가 제약을
  경계에 딱 붙여 푸는 것을 그렇게 우회하고 있었다. 여유는 지켜야 하는
  쪽을 깎는 게 아니라 만드는 쪽을 높여서 준다 — 이제 IK 만 IK_SLACK_M
  만큼 더 요구하고 계획기는 문턱을 그대로 지킨다.

           후보      경로 위 실제 최소 간격
  3link    23/25 -> 23/25    7.00 -> 10.89 mm
  램프      24/25 -> 19/25            10.04 mm

URDF 는 배달물 원본에 물성만 채운다
  예전에는 새로 지어서 스캔 메시가 AABB 상자로 퇴화하고, 파지 부위를
  뿌리로 다시 세운 트리가 나가고, 볼록분해 21조각이 버려졌다.
  배달물의 <inertial> 은 원래 밀도 1000 자리표시자였다 (link_1 441.02
  cm^3 -> 0.4410195 kg). 그 자리만 바꾸면 되는 구조였다.

  관성텐서도 고쳤다. Part.inertia_unit 에 메시 관성이 이미 있는데
  export 가 직육면체 공식을 쓰고 있었다. 굽은 팔은 관성적이 0 이 아니다.
  Drake 되읽기 오차 1e-10, 총질량 561.79 g = 396+84+82.

각도 허용 오차 3도 -> 5도, 후보 검사 창도 같이 넓힘
  통과 판정은 FoundationPose 가 읽은 각도로 한다. 창이 그 오차보다
  좁으면 작업자가 아무리 맞춰도 통과 못 하고 라운드가 무한 반복된다.

  창을 넓히면 실제 각도가 목표에서 그만큼 벗어난 채로 로봇이 움직인다.
  그래서 angle_probes 범위를 1.96σ 에서 1.96σ + 허용오차 로 넓혔다.
  한쪽만 고치면 검사한 적 없는 형상으로 로봇이 이동한다. 시뮬레이션은
  각도를 목표에 정확히 맞춰 주므로 이 구멍이 안 보인다.

수동 파지 — 시작 자세로 가기 전에 물체를 물린다
  begin() 이 팔을 시작 자세에 있다고 가정했다. 실물은 전원 켠 자리에
  있으므로, RRT 가 start_q -> start_q 를 풀어 경유점 하나를 내놓고
  드라이버가 계획에 없는 직선으로 팔을 보낸다. sync_from_robot() 이
  driver.joint_positions() 로 실제 자세를 읽는다.

  파지 단계 자체가 없었다 (시뮬은 물체가 그리퍼에 용접돼 있다).
  await_grasp(): 서보 끔 -> 물림 -> 확인 -> 서보 켬 -> 자세 재확인
  (꺼진 동안 처짐) -> 여유 검사 -> 그 다음 이동. 파지가 이동보다
  먼저여야 한다. 경로계획의 충돌 모형이 '물체를 든 팔' 이기 때문이다.

  hardware.RobotDriver 에 servo_on() 을 더했다. 끄기만 하는 인터페이스는
  덫이다 — 물린 뒤 다시 켤 방법이 없다.

my_work 정리 (figures/ outputs/ scratch/)
  파이썬 import 는 하나도 안 건드렸으므로 기존 실행 명령이 전부 그대로
  동작한다. 산출물이 다시 흩어지지 않도록 저장 경로도 함께 옮겼다.

PC 는 한 대면 된다
  robot_node.py 도 pydrake 를 쓰고 prepare() 를 돌리므로 "환경이 달라서
  나눈다" 는 이유가 성립하지 않는다. 무거운 FoundationPose 는 어차피
  별도 노드다. 2대로 나누면 prepare() 가 양쪽에서 각각 돌고, 플래그가
  다르면 두 쪽 장면이 조용히 달라진다.

검증: doctor 12/12, 3link 시뮬 전 과정 (23/25 후보, 2라운드 0.63% 수렴,
모든 이동에서 최소 간격 10.0mm, 순간이동·파고듦 0건), URDF 양쪽 경로
Drake 되읽기 통과.

Co-Authored-By: Claude Opus 5 (1M context) <noreply@anthropic.com>

File: my_work/outputs/estimated_3link.urdf (robot description, URDF)
Before this commit: robot 3link_estimated, 3 links, 2 joints
Links:
- link link0_base: mass 1.498054 -> 1.498432
- link link1_elbow: mass 0.269366 -> 0.332706
- link link2_tip: mass 0.104015 -> 0.154569
Joints:
- joint joint1: limit lower=0.000000 upper=2.967100 effort=10 velocity=1 -> lower=0.000000 upper=3.141593 effort=10 velocity=1
- joint joint2: limit lower=0.000000 upper=2.967100 effort=10 velocity=1 -> lower=0.000000 upper=3.141593 effort=10 velocity=1

Commit message: 연구 방향 검토 기록을 남긴다
논문 방향을 "정확한 asset 을 만든다" 에서 "추측 대신 측정한다" 로 옮기는
근거와, 그 과정에서 확인한 선행연구를 정리한다.

신규성 감사 결과는 정직하게 적었다. 정지 중력 측정이 질량과 무게중심만
준다는 것은 교과서 사실이고, 자세를 바꿔가며 분절 질량을 푸는 것은 생체역학의
반응판 기법으로 이미 있으며, D-최적 여기설계와 EIV/TLS 도 전부 기존 것이다.
새로운 것은 밀도 매개화가 그 한계를 "부위 개수의 상한" 으로 바꾼다는 귀결과,
자세 개수의 하한, 그리고 실측 기반 관절체 부위별 밀도를 재구성 자산에
기록하는 파이프라인이다.

재구성 오차가 무엇을 망가뜨리는지도 쟀다. 부피 오차는 질량에 그 절반쯤
들어오고(10% -> 6%), 도심 오차는 램프에서 1mm 에 2.4% 다. 그런데 라운드 수는
부피 오차 30% 에도 안 흔들린다 — 하한이 미지수 개수에서 나오기 때문이다.
그래서 이론 검증은 재구성 품질과 원리적으로 분리된다.

Co-Authored-By: Claude Opus 5 (1M context) <noreply@anthropic.com>

File: my_work/outputs/estimated_3link.urdf (robot description, URDF)
Before this commit: robot 3link_estimated, 3 links, 2 joints
Links:
- link link0_base: mass 1.498432 -> 1.498109
- link link1_elbow: mass 0.332706 -> 0.332922
- link link2_tip: mass 0.154569 -> 0.154505
